Commit message: URDF_pulgin_started

File: ballrobot/urdf/ballrobot.urdf (robot description, URDF)
Before this commit: robot ballrobot, 7 links, 6 joints
Links:
- added link robot_footprint; visual box size=0.001 0.001 0.001
Joints:
- added joint robot_footprint_joint: type fixed, parent robot_footprint, child base_link, origin xyz=0 0 0.04 rpy=3.14 3.14 0
